File: busdecoder.sch (KiCad schematic (older format))
At the start: 32 parts, among them SW1 SPST2P, SW3 SPST2P, U5 IC74HC00, U7 ESP32-S3FN8, Y2 40.000Mhz

Commit message: hw: RBL-XE schematic adapted to the C64 expansion port
Schematic sheets copied from VERA Module RBL-XE (2026-10-26 revision:
U19 ~OE gating with U24/U25, ESP32 strapping with ~ABUS_OE on GPIO 47,
open-drain IRQ U26, spare channels tied off), then the connector sheet
adapted to the Commodore 64:
- CART1/ECI1 (Atari) replaced by CART1 C64-EXPANSION-PORT, 2x22 edge
  fingers, 2.54 mm; /GAME, /EXROM, /ROML, /ROMH, /NMI, Dot Clock NC
- U6: /IO1 -> ~mIO1 -> GPIO 41, /IO2 -> ~mIO2 -> GPIO 42; BA, /DMA,
  /RESET to test points TP3, TP2, TP4
- U19 gating: U24 pin 4 = ~mIO1, pin 5 = 3V3 (were ~mEXSEL, ~mMPD)
- /RESET open-drain through U27 SN74LVC1G07 (+ C70), like the IRQ;
  U16 drives no C64 line, its spare inputs to GND (R78, R79, R80)
- VERA audio mix kept on TP5 (no audio pin on the C64 port)
- ~ATARI_RESET renamed ~C64_RESET, test points renumbered TP2-TP7

Netlist rebuilt and checked against the sheets with a connectivity
script (248 nets, no differences); cache library regenerated. The PCB
is still the Atari one and must be updated from the netlist.
Parts:
- added C67, C68: 100nF, Capacitor_SMD:C_0805_2012Metric_Pad1.18x1.45mm_HandSolder, symbol CCAP0805:100nF
- added R36, R53, R65, R70, R71: 10K, Resistor_SMD:R_0805_2012Metric_Pad1.20x1.40mm_HandSolder, symbol CRES0805:10K
- added U24, U25: SN74LVC00, Package_SO:TSSOP-14_4.4x5mm_P0.65mm, symbol RetroBitLab:SN74LVC00
- C25: value 100nF -> 1uF; symbol CCAP0805:100nF -> CCAP0805:1uF; LCSC C840116 -> C2798196
Connections:
- net ~mEXSEL is gone; now on net ~mIO1: U7.47 (MTDI)
- net ~mMPD is gone; now on net ~mIO2: U7.48 (MTMS)
- net 3V3: now also C67.1, C68.1, R36.2, R53.2, R65.2, R71.1, U24.14 (VCC), U24.5, U25.14 (VCC)
- net GND: now also C67.2, C68.2, R70.1, U24.7 (GND), U25.10, U25.12, U25.13, U25.7 (GND), U25.9
- net mPHI2: now also U25.4
- net mR~W: now also U24.1
- net ~mVCS0: now also R36.1, U24.2
- net ~ABUS_OE: now reaches U7.37 (SPICLK_P)
- net at U7.8 (GPIO3): now also R71.2
- net ~ATARI_RESET renamed ~C64_RESET
- net ~C64_RESET: now also R70.2
- net ~mCCTL renamed ~mIO2
- net ~mIO2: now also R65.1
- net ~mD1XX renamed ~mIO1
- net ~mIO1: now also R53.1, U24.4
- new net B: U25.3, U25.5
- new net a1: U24.8, U25.1
- new net a2: U24.11, U25.2
- new net n1: U24.10, U24.3, U24.9
- new net n2: U24.12, U24.13, U24.6
- new net ~OE: U25.6
Other:
- note added: "/IO1 ($DE00-$DEFF) -> GeoRAM window, data driven by the ESP32 (U19 enabled by /IO1)\n\n/IO2 $DF00-$DF1F and VERA selected through $DFFD -> mVCS0 (DEV_SEL_N) active\n\n/IO2 $DFFD/$DFFE/$DFFF -> VERA select latch, GeoRAM page/block (write only)"
- note added: "Accessing $DEXX (/IO1)"
- note added: "Accessing $DFXX (/IO2)"
- note added: "C64 Expansion Port Decoder:\n\n/IO1 GeoRAM window ($DE00-$DEFF),\n\n/IO2 VERA registers ($DF00-$DF1F), latch and GeoRAM registers ($DFFD-$DFFF)"
- note added: "C64 RESET IS ALWAYS ASSERTED\nWHEN POWERING UP THE MEMORY\nCONTROLLER"
- note added: "C64 SIGNALS ARE ALWAYS NOT VALIDATED\nWHEN POWERING UP THE MEMORY \nCONTROLLER AND THE SYSTEM CORE"
- note added: "VERA SELECT: latch $DFFD, software only"
- note removed: "Accessing $D1XX area space"
- note removed: "Accessing $D5XX area space"
- note removed: "PBI Bus Interface Decoder:\n\nI/O Space, Math Pack Disable, ROM ADDRESS ($D800-$DFFF),\n\nRAM PBI SPACE ($D600-$D7FF)"
- note removed: "PBI DEVICE ID: software selectable only"
- note removed: "When VERA Chip Select (mVCS0) latch is active & A15..A0 $D800-$DFFF -> MPD active (External 2K ROM)\n\nWhen VERA Chip Select (mVCS0) latch is active & A15..A0 $D600-$D7FF -> EXSEL active (External 512 bytes RAM)\n\nWhen access @ $D1xx and VERA Chip Select (mVCS0) latch is active -> EXSEL active"
- moved on the sheet: LD1, LD5, R32, R61
