File: cartridgeInterface.sch (KiCad schematic (older format))
At the start: 33 parts, among them U16 74LVC4245APW_118, U19 74LVC4245APW_118, U23 SN74HCT04DR, U3 74LVC4245APW_118, U4 74LVC4245APW_118, U6 74LVC4245APW_118

Commit message: hw: RBL-XE schematic adapted to the C64 expansion port
Schematic sheets copied from VERA Module RBL-XE (2026-10-26 revision:
U19 ~OE gating with U24/U25, ESP32 strapping with ~ABUS_OE on GPIO 47,
open-drain IRQ U26, spare channels tied off), then the connector sheet
adapted to the Commodore 64:
- CART1/ECI1 (Atari) replaced by CART1 C64-EXPANSION-PORT, 2x22 edge
  fingers, 2.54 mm; /GAME, /EXROM, /ROML, /ROMH, /NMI, Dot Clock NC
- U6: /IO1 -> ~mIO1 -> GPIO 41, /IO2 -> ~mIO2 -> GPIO 42; BA, /DMA,
  /RESET to test points TP3, TP2, TP4
- U19 gating: U24 pin 4 = ~mIO1, pin 5 = 3V3 (were ~mEXSEL, ~mMPD)
- /RESET open-drain through U27 SN74LVC1G07 (+ C70), like the IRQ;
  U16 drives no C64 line, its spare inputs to GND (R78, R79, R80)
- VERA audio mix kept on TP5 (no audio pin on the C64 port)
- ~ATARI_RESET renamed ~C64_RESET, test points renumbered TP2-TP7

Netlist rebuilt and checked against the sheets with a connectivity
script (248 nets, no differences); cache library regenerated. The PCB
is still the Atari one and must be updated from the netlist.
Parts:
- removed CART1: ATARI-CARTRIDGE, RetroBitLab:ATARI-LEFT-CARTRIDGE, symbol RetroBitLab:ATARI-CARTRIDGE
- removed ECI1: ECIBUS, RetroBitLab:ATARI-XE-ECI-SLOT, symbol RetroBitLab:ECIBUS
- removed R35, R36: 10K, Resistor_SMD:R_0805_2012Metric_Pad1.20x1.40mm_HandSolder, symbol CRES0805:10K
- removed mRD4: TestPoint, TestPoint:TestPoint_Pad_D2.0mm, symbol Connector:TestPoint
- added C66: 1uF, Capacitor_SMD:C_0805_2012Metric_Pad1.18x1.45mm_HandSolder, symbol CCAP0805:1uF
- added C69, C70: 100nF, Capacitor_SMD:C_0805_2012Metric_Pad1.18x1.45mm_HandSolder, symbol CCAP0805:100nF
- added CART1: C64-EXPANSION-PORT, RetroBitLab:C64-EXPANSION-CARTRIDGE, symbol RetroBitLab:C64-EXPANSION-PORT
- added R2, R6: 1K, Resistor_SMD:R_0805_2012Metric_Pad1.20x1.40mm_HandSolder, symbol CRES0805:1K
- added R72, R73, R74, R75, R76, R77, R78, R79, R80: CREZ08051%, Resistor_SMD:R_0805_2012Metric_Pad1.20x1.40mm_HandSolder, symbol CRES0805:CREZ08051%
- added U26, U27: SN74LVC1G07DBVR, Package_TO_SOT_SMD:SOT-23-5, symbol RetroBitLab:SN74LVC1G07DBVR
- R34, R7: value CREZ08051% -> 10K; symbol CRES0805:CREZ08051% -> CRES0805:10K; LCSC C328378 -> C84376
- renumbered ~mS5 to TP2, ~mS4 to TP3, ~mREF1 to TP4, ~mHALT1 to TP5, mRD5 to TP6, mD1XX1 to TP7
Connections:
- net ~REFRESH is gone; now on net ~RST: U6.9 (A6)
- net 3V3: now also R34.2, R7.2, U16.23 (VCCB), U19.23 (VCCB), U3.23 (VCCB), U4.23 (VCCB), U6.23 (VCCB), C69.1, C70.1, U26.5 (VCC), U27.5 (VCC)
- net 5V: now also CART1.2 (+5V), CART1.3 (+5V)
- net A0: now also CART1.Y (A0)
- net A1: now also CART1.X (A1)
- net A10: now also CART1.M (A10)
- net A11: now also CART1.L (A11)
- net A12: now also CART1.K (A12)
- net A13: now also CART1.J (A13)
- net A14: now also CART1.H (A14)
- net A15: now also CART1.F (A15)
- net A2: now also CART1.W (A2)
- net A3: now also CART1.V (A3)
- net A4: now also CART1.U (A4)
- net A5: now also CART1.T (A5)
- net A6: now also CART1.S (A6)
- net A7: now also CART1.R (A7)
- net A8: now also CART1.P (A8)
- net A9: now also CART1.N (A9)
- net AUDIO: now also TP5.1, C66.1
- net D0: now also CART1.21 (D0)
- net D1: now also CART1.20 (D1)
- net D2: now also CART1.19 (D2)
- net D3: now also CART1.18 (D3)
- net D4: now also CART1.17 (D4)
- net D5: now also CART1.16 (D5)
- net D6: now also CART1.15 (D6)
- net D7: now also CART1.14 (D7)
- net GND: now also U23.11, U23.13, U23.3, U23.5, U23.9, C69.2, C70.2, CART1.1 (GND), CART1.22 (GND), CART1.A (GND), CART1.Z (GND), R72.1, R73.1, R74.2, R75.1, R76.1, R77.1, R78.1, R79.1, R80.1, U26.3 (GND), U27.3 (GND); no longer R34.2, R7.2
- net PHI2: now also CART1.E (PHI2); no longer U23.3
- net R~W: now also CART1.5 (R/~W)
- net ~IRQ: now also CART1.4 (~IRQ), U26.4 (Y); no longer U16.6 (A3)
- net ~RST: now also CART1.C (~RESET), U27.4 (Y); no longer U16.9 (A6)
- net ~mVIRQ: now also U26.2 (A); no longer U16.18 (B3)
- net ~ABUS_OE: now reaches R34.1, U4.22 (~OE)
- net ~ABUS_OE: now also R7.1, U3.22 (~OE)
- net at U16.14 (B7): now also R72.2
- net at U6.10 (A7): now also R74.1
- net at U23.4: no longer U19.22 (~OE)
- net RD4: no longer names the net of U16.4 (A1)
- net RD5: no longer names the net of U16.3 (A0)
- net mRD4: no longer names the net of U16.20 (B1)
- net mRD4: now also R76.2
- net mRD5: no longer names the net of U16.21 (B0)
- net mRD5: now also R77.2; no longer TP6.1
- net mREFRESH renamed ~mRST
- net ~ATARI_RESET: no longer names the net of U16.15 (B6)
- net ~ATARI_RESET: now also R75.2
- net ~CCTL renamed ~IO2
- net ~IO2: now also CART1.10 (~IO2)
- net ~D1XX renamed ~IO1
- net ~IO1: now also CART1.7 (~IO1)
- net ~EXSEL: no longer names the net of U16.7 (A4)
- net ~HALT: no longer names the net of U16.5 (A2)
- net ~MPD: no longer names the net of U16.8 (A5)
- net ~S4 renamed BA
- net BA: now also CART1.12 (BA)
- net ~S5 renamed ~DMA
- net ~DMA: now also CART1.13 (~DMA)
- net ~mCCTL renamed ~mIO2
- net ~mIO2: now also TP6.1
- net ~mD1XX renamed ~mIO1
- net ~mEXSEL: no longer names the net of U16.17 (B4)
- net ~mEXSEL: now also R79.2
- net ~mHALT: no longer names the net of U16.19 (B2)
- net ~mHALT: now also R73.2; no longer TP5.1
- net ~mMPD: no longer names the net of U16.16 (B5)
- net ~mMPD: now also R80.2
- net ~mS4 renamed mBA
- net ~mS5 renamed ~mDMA
- new net: R78.2, U16.18 (B3)
- new net: C66.2, R2.1, R6.1
- new net AUD1L: R2.2
- new net AUD1R: R6.2
- new net ~C64_RESET: U27.2 (A)
- new net ~OE: U19.22 (~OE)
- no-connect marks 18 -> 20
Other:
- note added: "AUDIO MIXER (NO AUDIO PIN ON THE C64 PORT: TP5)"
- note added: "C64 /RESET\nopen-drain"
- note added: "COMMODORE 64 EXPANSION PORT INTERFACE"
- note added: "Interrupt Setup\nbetween VERA & CPU"
- note added: "TEST POINTS"
- note removed: "ATARI 130XE ECI & CARTRIDGE INTERFACE"
- note removed: "AUDIO MIXER INSIDE ATARI"
- note removed: "UNCONNECTED IN THIS PROJECT"
- moved on the sheet: U23B
