File: powersupply.sch (KiCad schematic (older format))
At the start: 42 parts, among them J4 DX07S016JA1R1500, J5 PJ-002AH-SMT-TR, Q3 BC817,SOT-23, Q4 BC817,SOT-23, U12 USBCH340T, U13 AMS1117-3.3, U14 AMS1117-1.2, U15 L7805, U17 MAX40200AUK, U18 MAX40200AUK, Y1 12MHzC

Commit message: hw: RBL-XE schematic adapted to the C64 expansion port
Schematic sheets copied from VERA Module RBL-XE (2026-10-26 revision:
U19 ~OE gating with U24/U25, ESP32 strapping with ~ABUS_OE on GPIO 47,
open-drain IRQ U26, spare channels tied off), then the connector sheet
adapted to the Commodore 64:
- CART1/ECI1 (Atari) replaced by CART1 C64-EXPANSION-PORT, 2x22 edge
  fingers, 2.54 mm; /GAME, /EXROM, /ROML, /ROMH, /NMI, Dot Clock NC
- U6: /IO1 -> ~mIO1 -> GPIO 41, /IO2 -> ~mIO2 -> GPIO 42; BA, /DMA,
  /RESET to test points TP3, TP2, TP4
- U19 gating: U24 pin 4 = ~mIO1, pin 5 = 3V3 (were ~mEXSEL, ~mMPD)
- /RESET open-drain through U27 SN74LVC1G07 (+ C70), like the IRQ;
  U16 drives no C64 line, its spare inputs to GND (R78, R79, R80)
- VERA audio mix kept on TP5 (no audio pin on the C64 port)
- ~ATARI_RESET renamed ~C64_RESET, test points renumbered TP2-TP7

Netlist rebuilt and checked against the sheets with a connectivity
script (248 nets, no differences); cache library regenerated. The PCB
is still the Atari one and must be updated from the netlist.
Parts:
- R56: value 0R -> CREZ08051%; symbol CRES0805:0R -> CRES0805:CREZ08051%
Changed lines of the file:
@@
 Sheet 6 7
 Title "POWERSUPPLY and USB"
-Date "2026-09-01"
+Date "2026-10-26"
 Rev "1.0"
 Comp "RetroBit Lab"
@@
 $EndComp
 $Comp
-L CRES0805:0R R56
+L CRES0805:CREZ08051% R56
 U 1 1 68B89F7F
 P 3720 4940
 F 0 "R56" V 3645 4940 50  0000 C CNN
-F 1 "0R" V 3795 4935 50  0000 C CNN
+F 1 "CREZ08051%" V 3795 4935 50  0000 C CNN
 F 2 "Resistor_SMD:R_0805_2012Metric_Pad1.20x1.40mm_HandSolder" H 3720 4940 50  0001 C CNN
-F 3 "https://www.lcsc.com/datasheet/C328378.pdf" H 3720 4940 50  0001 C CNN
+F 3 "https://www.lcsc.com/datasheet/C328378.pdf?spm=wm.sxq.inf.ggs&lcsc_vid=QAIPVVVVRlJXV1FQQABeBQAAQQNaVFMAR1IIXwYHFlgxVlNfRFFfVlJfTlRXVDsOAxUeFF5JWBYZEEoKFBINSQcJGk4%3D" H 3720 4940 50  0001 C CNN
 F 4 "C328378" H 3720 4940 50  0001 C CNN "LCSC"
 	1    3720 4940
