File: vga-analog.sch (KiCad schematic (older format))
At the start: 27 parts, among them J1 CONN_SMD_HEADER_BOX_02x08_Odd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, J2 DS1038-15FBNSiA74-0CC

Commit message: hw: RBL-XE schematic adapted to the C64 expansion port
Schematic sheets copied from VERA Module RBL-XE (2026-10-26 revision:
U19 ~OE gating with U24/U25, ESP32 strapping with ~ABUS_OE on GPIO 47,
open-drain IRQ U26, spare channels tied off), then the connector sheet
adapted to the Commodore 64:
- CART1/ECI1 (Atari) replaced by CART1 C64-EXPANSION-PORT, 2x22 edge
  fingers, 2.54 mm; /GAME, /EXROM, /ROML, /ROMH, /NMI, Dot Clock NC
- U6: /IO1 -> ~mIO1 -> GPIO 41, /IO2 -> ~mIO2 -> GPIO 42; BA, /DMA,
  /RESET to test points TP3, TP2, TP4
- U19 gating: U24 pin 4 = ~mIO1, pin 5 = 3V3 (were ~mEXSEL, ~mMPD)
- /RESET open-drain through U27 SN74LVC1G07 (+ C70), like the IRQ;
  U16 drives no C64 line, its spare inputs to GND (R78, R79, R80)
- VERA audio mix kept on TP5 (no audio pin on the C64 port)
- ~ATARI_RESET renamed ~C64_RESET, test points renumbered TP2-TP7

Netlist rebuilt and checked against the sheets with a connectivity
script (248 nets, no differences); cache library regenerated. The PCB
is still the Atari one and must be updated from the netlist.
Connections:
- net AUDIOL renamed AUD1L
- net AUDIOR renamed AUD1R
Changed lines of the file:
@@
 Sheet 7 7
 Title "VGA ANALOG AND EXTERNAL VIDEO CONNECTOR"
-Date "2026-09-01"
+Date "2026-10-26"
 Rev "1.0"
 Comp "RetroBit Lab"
@@
 EXTERNAL VIDEO CONNECTOR
 Text GLabel 4890 5715 0    39   Input ~ 0
-AUDIOL
+AUD1L
 Text GLabel 5510 5715 2    39   Input ~ 0
-AUDIOR
+AUD1R
 Wire Wire Line
 	4890 5715 4950 5715
