File: vera-fpga-flash.sch (KiCad schematic (older format))
At the start: 31 parts, among them J3 CONN_DM3AT-SF-PEJM5, J7 SJ-3523-SMT-TR, U10 W25Q16JVSNIQ, U11 WM8524CGEDT, U8 74CBTLV3126PW,118, U9 CD4011B

Commit message: hw: RBL-XE schematic adapted to the C64 expansion port
Schematic sheets copied from VERA Module RBL-XE (2026-10-26 revision:
U19 ~OE gating with U24/U25, ESP32 strapping with ~ABUS_OE on GPIO 47,
open-drain IRQ U26, spare channels tied off), then the connector sheet
adapted to the Commodore 64:
- CART1/ECI1 (Atari) replaced by CART1 C64-EXPANSION-PORT, 2x22 edge
  fingers, 2.54 mm; /GAME, /EXROM, /ROML, /ROMH, /NMI, Dot Clock NC
- U6: /IO1 -> ~mIO1 -> GPIO 41, /IO2 -> ~mIO2 -> GPIO 42; BA, /DMA,
  /RESET to test points TP3, TP2, TP4
- U19 gating: U24 pin 4 = ~mIO1, pin 5 = 3V3 (were ~mEXSEL, ~mMPD)
- /RESET open-drain through U27 SN74LVC1G07 (+ C70), like the IRQ;
  U16 drives no C64 line, its spare inputs to GND (R78, R79, R80)
- VERA audio mix kept on TP5 (no audio pin on the C64 port)
- ~ATARI_RESET renamed ~C64_RESET, test points renumbered TP2-TP7

Netlist rebuilt and checked against the sheets with a connectivity
script (248 nets, no differences); cache library regenerated. The PCB
is still the Atari one and must be updated from the netlist.
Parts:
- added R35: CREZ08051%, Resistor_SMD:R_0805_2012Metric_Pad1.20x1.40mm_HandSolder, symbol CRES0805:CREZ08051%
Connections:
- net 3V3: now also R35.1; no longer U11.11 (~MUTE), U11.12 (AIFMODE)
- net AUD1L: now reaches R67.1
- net AUD1L: now also J7.3 (RING); no longer J7.2 (TIP)
- net AUD1R: now reaches R68.1
- net AUD1R: now also J7.2 (TIP); no longer J7.3 (RING)
- net AUDIOL: no longer names the net of C31.1, R45.1, R67.2
- net AUDIOR: no longer names the net of C30.1, R46.1, R68.2
- new net: R35.2, U11.11 (~MUTE), U11.12 (AIFMODE)
Other:
- moved on the sheet: R67, R68
Changed lines of the file:
@@
 Sheet 5 7
 Title "uSD Card, FPGA FLASH and AUDIO SECTION"
-Date "2026-09-01"
+Date "2026-10-26"
 Rev "1.0"
 Comp "RetroBit Lab"
@@
 	3300 5210 3300 5240
 Connection ~ 3300 5210
-Text GLabel 4050 5110 2    39   Output ~ 0
-AUDIOL
-Wire Wire Line
-	3300 5210 4050 5210
-Text GLabel 4050 5210 2    39   Output ~ 0
-AUDIOR
 Text Label 3240 2645 0    39   ~ 0
 SD_SSEL_N
@@
 Wire Wire Line
 	1325 6010 960  6010
-Text GLabel 1035 5685 2    39   BiDi ~ 0
+Text GLabel 1035 5570 2    39   BiDi ~ 0
 3V3
 Wire Wire Line
-	1035 5685 960  5685
+	1035 5570 960  5570
 Wire Wire Line
 	1325 5910 960  5910
@@
 Text Label 5565 1060 2    39   ~ 0
 SD_SSEL_N
-Wire Wire Line
-	960  5685 960  5910
-Connection ~ 960  5910
 $Comp
 L RetroBitLab:SJ-3523-SMT-TR J7
@@
 	-1   0    0    1
 $EndComp
-Text GLabel 5085 5665 0    39   Input ~ 0
-AUDIOL
-Text GLabel 5095 5965 0    39   Input ~ 0
-AUDIOR
+Text GLabel 5525 5965 0    39   Input ~ 0
+AUD1L
+Text GLabel 5520 5665 0    39   Input ~ 0
+AUD1R
 $Comp
 L power:GND #PWR03
@@
 $EndComp
 Wire Wire Line
-	5570 5665 5440 5665
-Wire Wire Line
-	5570 5965 5450 5965
+	5015 5110 4885 5110
 Wire Wire Line
 	5570 6065 5525 6065
 Wire Wire Line
 	5525 6065 5525 6105
-Text Notes 5135 5370 0    79   Italic 16
+Text Notes 5340 5500 0    79   Italic 16
 AUDIO 3.5mm OUTPUT
 Text Notes 3515 7405 0    118  ~ 24
@@
 L CRES0805:560R R67
 U 1 1 68CDB550
-P 5345 5665
-F 0 "R67" V 5410 5665 50  0000 C CNN
-F 1 "560R" V 5275 5670 50  0000 C CNN
-F 2 "Resistor_SMD:R_0805_2012Metric_Pad1.20x1.40mm_HandSolder" H 5345 5665 50  0001 C CNN
-F 3 "https://lcsc.com/datasheet/lcsc_datasheet_2411221126_UNI-ROYAL-0805W8F4700T5E_C17710.pdf" H 5345 5665 50  0001 C CNN
-F 4 "C28636" H 5345 5665 50  0001 C CNN "LCSC"
-	1    5345 5665
+P 4790 5110
+F 0 "R67" V 4855 5110 50  0000 C CNN
+F 1 "560R" V 4720 5115 50  0000 C CNN
+F 2 "Resistor_SMD:R_0805_2012Metric_Pad1.20x1.40mm_HandSolder" H 4790 5110 50  0001 C CNN
+F 3 "https://lcsc.com/datasheet/lcsc_datasheet_2411221126_UNI-ROYAL-0805W8F4700T5E_C17710.pdf" H 4790 5110 50  0001 C CNN
+F 4 "C28636" H 4790 5110 50  0001 C CNN "LCSC"
+	1    4790 5110
 	0    1    1    0
 $EndComp
-$Comp
-L CRES0805:560R R68
-U 1 1 68CDE7A1
-P 5355 5965
-F 0 "R68" V 5420 5965 50  0000 C CNN
-F 1 "560R" V 5285 5970 50  0000 C CNN
-F 2 "Resistor_SMD:R_0805_2012Metric_Pad1.20x1.40mm_HandSolder" H 5355 5965 50  0001 C CNN
-F 3 "https://lcsc.com/datasheet/lcsc_datasheet_2411221126_UNI-ROYAL-0805W8F4700T5E_C17710.pdf" H 5355 5965 50  0001 C CNN
-F 4 "C28636" H 5355 5965 50  0001 C CNN "LCSC"
-	1    5355 5965
-	0    1    1    0
-$EndComp
-Wire Wire Line
-	5240 5665 5085 5665
-Wire Wire Line
-	5250 5965 5095 5965
 $Comp
 L RetroBitLab:CD4011B U9
@@
 Connection ~ 3800 5110
 Wire Wire Line
-	3800 5110 4050 5110
-Wire Wire Line
 	3800 5440 3800 5485
 Wire Wire Line
@@
 $EndComp
 Connection ~ 3225 6010
+$Comp
+L CRES0805:560R R68
+U 1 1 68CDE7A1
+P 4310 5210
+F 0 "R68" V 4375 5210 50  0000 C CNN
+F 1 "560R" V 4240 5215 50  0000 C CNN
+F 2 "Resistor_SMD:R_0805_2012Metric_Pad1.20x1.40mm_HandSolder" H 4310 5210 50  0001 C CNN
+F 3 "https://lcsc.com/datasheet/lcsc_datasheet_2411221126_UNI-ROYAL-0805W8F4700T5E_C17710.pdf" H 4310 5210 50  0001 C CNN
+F 4 "C28636" H 4310 5210 50  0001 C CNN "LCSC"
+	1    4310 5210
+	0    1    1    0
+$EndComp
+Wire Wire Line
+	3300 5210 4205 5210
+Wire Wire Line
+	3800 5110 4685 5110
+Wire Wire Line
+	4405 5210 5020 5210
+Wire Wire Line
+	5520 5665 5570 5665
+Wire Wire Line
+	5525 5965 5570 5965
+Text GLabel 5020 5210 2    39   Output ~ 0
+AUD1R
+Text GLabel 5015 5110 2    39   Output ~ 0
+AUD1L
+$Comp
+L CRES0805:CREZ08051% R35
+U 1 1 6ADC11D2
+P 960 5725
+F 0 "R35" H 1005 5715 50  0000 L CNN
+F 1 "CREZ08051%" V 870 5470 50  0000 L CNN
+F 2 "Resistor_SMD:R_0805_2012Metric_Pad1.20x1.40mm_HandSolder" H 960 5725 50  0001 C CNN
+F 3 "https://www.lcsc.com/datasheet/C328378.pdf?spm=wm.sxq.inf.ggs&lcsc_vid=QAIPVVVVRlJXV1FQQABeBQAAQQNaVFMAR1IIXwYHFlgxVlNfRFFfVlJfTlRXVDsOAxUeFF5JWBYZEEoKFBINSQcJGk4%3D" H 960 5725 50  0001 C CNN
+F 4 "C328378" H 960 5725 50  0001 C CNN "LCSC"
+	1    960  5725
+	1    0    0    -1
+$EndComp
+Wire Wire Line
+	960  5570 960  5630
+Wire Wire Line
+	960  5830 960  5910
+Connection ~ 960  5910
 $EndSCHEMATC

Commit message: hw: C36, R37-R44, J7, X1 to the parts used on RBL-XE
C36 C377773, R37-R44 C17713 (JLCPCB Basic), J7 PJ-313D C668608,
X1 YXC OT3EL89CJI-111YLC-25M C7471623: the old ones are out of stock or
short at JLCPCB. The J7 footprint still has to be changed on the PCB.
Parts:
- C36: symbol CCAP0805:2.2uF -> CCAP0805:2.2uF-X5R; LCSC C7393943 -> C377773
- J7: value SJ-3523-SMT-TR -> PJ-313D; footprint RetroBitLab:CONN_AUDIO_CUI_SJ-3523-SMT-TR -> RetroBitLab:jack_3.5_pj313d-smt; symbol RetroBitLab:SJ-3523-SMT-TR -> RetroBitLab:CONN_AUDIO_JACK_3.5_PJ313D; Availability In Stock -> (none); Check_prices https://www.snapeda.com/parts/SJ-3523-SMT-TR/Same+Sky/view-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 -> (none); Description \\n \\n 3.5 mm, Stereo, Right Angle, Surface Mount (SMT), 3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 -> (none); LCSC C4991872 -> C668608; MANUFACTURER CUI Inc -> (none); MF Same Sky -> SHOU HAN; MP SJ-3523-SMT-TR -> PJ-313D; Package None -> (none); Price None -> (none); SnapEDA_Link https://www.snapeda.com/parts/SJ-3523-SMT-TR/Same+Sky/view-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 -> (none)
- R37, R38, R39, R40, R41, R42, R43, R44: symbol CRES0805:47K -> CRES0805:47K-125mW; LCSC C20142780 -> C17713
Changed lines of the file:
@@
 $EndComp
 $Comp
-L CRES0805:47K R43
+L CRES0805:47K-125mW R43
 U 1 1 68B76F19
 P 10640 4815
@@
 F 1 "47K" V 10575 4805 50  0000 C CNN
 F 2 "Resistor_SMD:R_0805_2012Metric_Pad1.20x1.40mm_HandSolder" H 10640 4815 50  0001 C CNN
-F 3 "https://www.lcsc.com/datasheet/C20142780.pdf" H 10640 4815 50  0001 C CNN
-F 4 "C20142780" H 10640 4815 50  0001 C CNN "LCSC"
+F 3 "https://www.lcsc.com/datasheet/C17713.pdf" H 10640 4815 50  0001 C CNN
+F 4 "C17713" H 10640 4815 50  0001 C CNN "LCSC"
 	1    10640 4815
 	0    1    1    0
 $EndComp
 $Comp
-L CRES0805:47K R44
+L CRES0805:47K-125mW R44
 U 1 1 68B7750F
 P 10640 5115
@@
 F 1 "47K" V 10570 5110 50  0000 C CNN
 F 2 "Resistor_SMD:R_0805_2012Metric_Pad1.20x1.40mm_HandSolder" H 10640 5115 50  0001 C CNN
-F 3 "https://www.lcsc.com/datasheet/C20142780.pdf" H 10640 5115 50  0001 C CNN
-F 4 "C20142780" H 10640 5115 50  0001 C CNN "LCSC"
+F 3 "https://www.lcsc.com/datasheet/C17713.pdf" H 10640 5115 50  0001 C CNN
+F 4 "C17713" H 10640 5115 50  0001 C CNN "LCSC"
 	1    10640 5115
 	0    1    1    0
@@
 $EndComp
 $Comp
-L CRES0805:47K R37
+L CRES0805:47K-125mW R37
 U 1 1 68CF6C3B
 P 7340 1330
@@
 F 1 "47K" H 7399 1280 50  0000 L CNN
 F 2 "Resistor_SMD:R_0805_2012Metric_Pad1.20x1.40mm_HandSolder" H 7340 1330 50  0001 C CNN
-F 3 "https://www.lcsc.com/datasheet/C20142780.pdf" H 7340 1330 50  0001 C CNN
-F 4 "C20142780" H 7340 1330 50  0001 C CNN "LCSC"
+F 3 "https://www.lcsc.com/datasheet/C17713.pdf" H 7340 1330 50  0001 C CNN
+F 4 "C17713" H 7340 1330 50  0001 C CNN "LCSC"
 	1    7340 1330
 	1    0    0    -1
 $EndComp
 $Comp
-L CRES0805:47K R38
+L CRES0805:47K-125mW R38
 U 1 1 68D00370
 P 7590 1330
@@
 F 1 "47K" H 7649 1280 50  0000 L CNN
 F 2 "Resistor_SMD:R_0805_2012Metric_Pad1.20x1.40mm_HandSolder" H 7590 1330 50  0001 C CNN
-F 3 "https://www.lcsc.com/datasheet/C20142780.pdf" H 7590 1330 50  0001 C CNN
-F 4 "C20142780" H 7590 1330 50  0001 C CNN "LCSC"
+F 3 "https://www.lcsc.com/datasheet/C17713.pdf" H 7590 1330 50  0001 C CNN
+F 4 "C17713" H 7590 1330 50  0001 C CNN "LCSC"
 	1    7590 1330
 	1    0    0    -1
 $EndComp
 $Comp
-L CRES0805:47K R39
+L CRES0805:47K-125mW R39
 U 1 1 68D00935
 P 7840 1330
@@
 F 1 "47K" H 7899 1280 50  0000 L CNN
 F 2 "Resistor_SMD:R_0805_2012Metric_Pad1.20x1.40mm_HandSolder" H 7840 1330 50  0001 C CNN
-F 3 "https://www.lcsc.com/datasheet/C20142780.pdf" H 7840 1330 50  0001 C CNN
-F 4 "C20142780" H 7840 1330 50  0001 C CNN "LCSC"
+F 3 "https://www.lcsc.com/datasheet/C17713.pdf" H 7840 1330 50  0001 C CNN
+F 4 "C17713" H 7840 1330 50  0001 C CNN "LCSC"
 	1    7840 1330
 	1    0    0    -1
 $EndComp
 $Comp
-L CRES0805:47K R40
+L CRES0805:47K-125mW R40
 U 1 1 68D00E4E
 P 8090 1330
@@
 F 1 "47K" H 8149 1280 50  0000 L CNN
 F 2 "Resistor_SMD:R_0805_2012Metric_Pad1.20x1.40mm_HandSolder" H 8090 1330 50  0001 C CNN
-F 3 "https://www.lcsc.com/datasheet/C20142780.pdf" H 8090 1330 50  0001 C CNN
-F 4 "C20142780" H 8090 1330 50  0001 C CNN "LCSC"
+F 3 "https://www.lcsc.com/datasheet/C17713.pdf" H 8090 1330 50  0001 C CNN
+F 4 "C17713" H 8090 1330 50  0001 C CNN "LCSC"
 	1    8090 1330
 	1    0    0    -1
 $EndComp
 $Comp
-L CRES0805:47K R41
+L CRES0805:47K-125mW R41
 U 1 1 68D0121B
 P 8340 1330
@@
 F 1 "47K" H 8399 1280 50  0000 L CNN
 F 2 "Resistor_SMD:R_0805_2012Metric_Pad1.20x1.40mm_HandSolder" H 8340 1330 50  0001 C CNN
-F 3 "https://www.lcsc.com/datasheet/C20142780.pdf" H 8340 1330 50  0001 C CNN
-F 4 "C20142780" H 8340 1330 50  0001 C CNN "LCSC"
+F 3 "https://www.lcsc.com/datasheet/C17713.pdf" H 8340 1330 50  0001 C CNN
+F 4 "C17713" H 8340 1330 50  0001 C CNN "LCSC"
 	1    8340 1330
 	1    0    0    -1
@@
 	2600 5435 2600 5510
 $Comp
-L CRES0805:47K R42
+L CRES0805:47K-125mW R42
 U 1 1 68E055B4
 P 8090 2780
@@
 F 1 "47K" H 8149 2730 50  0000 L CNN
 F 2 "Resistor_SMD:R_0805_2012Metric_Pad1.20x1.40mm_HandSolder" H 8090 2780 50  0001 C CNN
-F 3 "https://www.lcsc.com/datasheet/C20142780.pdf" H 8090 2780 50  0001 C CNN
-F 4 "C20142780" H 8090 2780 50  0001 C CNN "LCSC"
+F 3 "https://www.lcsc.com/datasheet/C17713.pdf" H 8090 2780 50  0001 C CNN
+F 4 "C17713" H 8090 2780 50  0001 C CNN "LCSC"
 	1    8090 2780
 	1    0    0    -1
@@
 SD_SSEL_N
 $Comp
-L RetroBitLab:SJ-3523-SMT-TR J7
+L RetroBitLab:CONN_AUDIO_JACK_3.5_PJ313D J7
 U 1 1 6912EA11
 P 5970 5865
 F 0 "J7" H 5342 5806 50  0000 R CNN
-F 1 "SJ-3523-SMT-TR" H 6165 6180 50  0000 R CNN
-F 2 "RetroBitLab:CONN_AUDIO_CUI_SJ-3523-SMT-TR" H 5970 5865 50  0001 L BNN
-F 3 "https://www.lcsc.com/datasheet/C4991872.pdf" H 5970 5865 50  0001 L BNN
-F 4 "Same Sky" H 5970 5865 50  0001 L BNN "MF"
-F 5 "\\n                        \\n                            3.5 mm, Stereo, Right Angle, Surface Mount (SMT), 3 Conductors, 0 Internal Switches, Audio Jack Connector\\n                        \\n" H 5970 5865 50  0001 L BNN "Description"
-F 6 "None" H 5970 5865 50  0001 L BNN "Package"
-F 7 "None" H 5970 5865 50  0001 L BNN "Price"
-F 8 "https://www.snapeda.com/parts/SJ-3523-SMT-TR/Same+Sky/view-part/?ref=eda" H 5970 5865 50  0001 L BNN "Check_prices"
-F 9 "https://www.snapeda.com/parts/SJ-3523-SMT-TR/Same+Sky/view-part/?ref=snap" H 5970 5865 50  0001 L BNN "SnapEDA_Link"
-F 10 "SJ-3523-SMT-TR" H 5970 5865 50  0001 L BNN "MP"
-F 11 "In Stock" H 5970 5865 50  0001 L BNN "Availability"
-F 12 "CUI Inc" H 5970 5865 50  0001 L BNN "MANUFACTURER"
-F 13 "C4991872" H 5970 5865 50  0001 C CNN "LCSC"
+F 1 "PJ-313D" H 6165 6180 50  0000 R CNN
+F 2 "RetroBitLab:jack_3.5_pj313d-smt" H 5970 5865 50  0001 L BNN
+F 3 "https://www.lcsc.com/datasheet/C668608.pdf" H 5970 5865 50  0001 L BNN
+F 4 "SHOU HAN" H 5970 5865 50  0001 L BNN "MF"
+F 5 "PJ-313D" H 5970 5865 50  0001 L BNN "MP"
+F 6 "C668608" H 5970 5865 50  0001 C CNN "LCSC"
 	1    5970 5865
 	-1   0    0    1
@@
 	2745 6535 2745 6610
 $Comp
-L CCAP0805:2.2uF C36
+L CCAP0805:2.2uF-X5R C36
 U 1 1 68B87B28
 P 2750 6435
@@
 F 1 "2.2uF" H 2842 6390 50  0000 L CNN
 F 2 "Capacitor_SMD:C_0805_2012Metric_Pad1.18x1.45mm_HandSolder" H 2755 6435 50  0001 C CNN
-F 3 "https://lcsc.com/datasheet/lcsc_datasheet_2410121534_CCTC-TCC0805X7R225M500FT_C7393943.pdf" H 2755 6435 50  0001 C CNN
-F 4 "C7393943" H 2750 6435 50  0001 C CNN "LCSC"
+F 3 "https://www.lcsc.com/datasheet/C377773.pdf" H 2755 6435 50  0001 C CNN
+F 4 "C377773" H 2750 6435 50  0001 C CNN "LCSC"
 	1    2750 6435
 	1    0    0    -1
