File: vera-fpga.sch (KiCad schematic (older format))
At the start: 22 parts, among them J6 CONN_SMD_01x08_Staggered_2.54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, Q1 MOSFET-BSS138-SOT-23, U2 ICE40UP5K-SG48ITR, X1 ECS-2033-250-BN

Commit message: hw: RBL-XE schematic adapted to the C64 expansion port
Schematic sheets copied from VERA Module RBL-XE (2026-10-26 revision:
U19 ~OE gating with U24/U25, ESP32 strapping with ~ABUS_OE on GPIO 47,
open-drain IRQ U26, spare channels tied off), then the connector sheet
adapted to the Commodore 64:
- CART1/ECI1 (Atari) replaced by CART1 C64-EXPANSION-PORT, 2x22 edge
  fingers, 2.54 mm; /GAME, /EXROM, /ROML, /ROMH, /NMI, Dot Clock NC
- U6: /IO1 -> ~mIO1 -> GPIO 41, /IO2 -> ~mIO2 -> GPIO 42; BA, /DMA,
  /RESET to test points TP3, TP2, TP4
- U19 gating: U24 pin 4 = ~mIO1, pin 5 = 3V3 (were ~mEXSEL, ~mMPD)
- /RESET open-drain through U27 SN74LVC1G07 (+ C70), like the IRQ;
  U16 drives no C64 line, its spare inputs to GND (R78, R79, R80)
- VERA audio mix kept on TP5 (no audio pin on the C64 port)
- ~ATARI_RESET renamed ~C64_RESET, test points renumbered TP2-TP7

Netlist rebuilt and checked against the sheets with a connectivity
script (248 nets, no differences); cache library regenerated. The PCB
is still the Atari one and must be updated from the netlist.
Parts:
- removed R65: 10K, Resistor_SMD:R_0805_2012Metric_Pad1.20x1.40mm_HandSolder, symbol CRES0805:10K
- JP1, JP3: footprint (none) -> Jumper:SolderJumper-2_P1.3mm_Open_RoundedPad1.0x1.5mm
Changed lines of the file:
@@
 Sheet 2 7
 Title "VERA MODULE AND PROGRAMMING CONNECTOR"
-Date "2026-09-01"
+Date "2026-10-26"
 Rev "1.0"
 Comp "RetroBit Lab"
@@
 Text GLabel 1990 2800 0    39   Input ~ 0
 ~mWE
-Text GLabel 1400 2900 0    39   Input ~ 0
+Text GLabel 1400 2900 0    39   Output ~ 0
 ~mVIRQ
 Text GLabel 1990 3000 0    39   Input ~ 0
@@
 	1    0    0    -1
 $EndComp
-$Comp
-L CRES0805:10K R65
-U 1 1 68CF9E81
-P 1570 2525
-F 0 "R65" H 1629 2566 50  0000 L CNN
-F 1 "10K" H 1629 2475 50  0000 L CNN
-F 2 "Resistor_SMD:R_0805_2012Metric_Pad1.20x1.40mm_HandSolder" H 1570 2525 50  0001 C CNN
-F 3 "https://lcsc.com/datasheet/lcsc_datasheet_2506161110_YAGEO-RC0805FR-0710KL_C84376.pdf" H 1570 2525 50  0001 C CNN
-F 4 "C84376" H 1570 2525 50  0001 C CNN "LCSC"
-	1    1570 2525
-	1    0    0    -1
-$EndComp
-Text GLabel 1465 2135 0    50   BiDi ~ 0
-3V3
-Wire Wire Line
-	1465 2135 1570 2135
-Wire Wire Line
-	1570 2135 1570 2430
-Wire Wire Line
-	1570 2900 2190 2900
-Wire Wire Line
-	1570 2630 1570 2900
-Wire Wire Line
-	1570 2900 1400 2900
-Connection ~ 1570 2900
 Text GLabel 8410 1090 0    50   BiDi ~ 0
 5V
@@
 F 0 "JP1" V 8480 1338 50  0000 L CNN
 F 1 "SolderJumper_2_Open" V 8525 1338 50  0001 L CNN
-F 2 "" H 8480 1270 50  0001 C CNN
+F 2 "Jumper:SolderJumper-2_P1.3mm_Open_RoundedPad1.0x1.5mm" H 8480 1270 50  0001 C CNN
 F 3 "~" H 8480 1270 50  0001 C CNN
 	1    8480 1270
@@
 F 0 "JP3" V 8980 1338 50  0000 L CNN
 F 1 "SolderJumper_2_Open" V 9025 1338 50  0001 L CNN
-F 2 "" H 8980 1270 50  0001 C CNN
+F 2 "Jumper:SolderJumper-2_P1.3mm_Open_RoundedPad1.0x1.5mm" H 8980 1270 50  0001 C CNN
 F 3 "~" H 8980 1270 50  0001 C CNN
 	1    8980 1270
@@
 Wire Wire Line
 	8480 1090 8480 1120
+Wire Wire Line
+	1400 2900 2190 2900
 $EndSCHEMATC

Commit message: hw: C36, R37-R44, J7, X1 to the parts used on RBL-XE
C36 C377773, R37-R44 C17713 (JLCPCB Basic), J7 PJ-313D C668608,
X1 YXC OT3EL89CJI-111YLC-25M C7471623: the old ones are out of stock or
short at JLCPCB. The J7 footprint still has to be changed on the PCB.
Parts:
- X1: value ECS-2033-250-BN -> OT3EL89CJI-111YLC-25M; LCSC C2441279 -> C7471623; MANUFACTURER ECS Inc -> YXC; PARTREV 11/15/13 -> (none); STANDARD Manufacturer Recommendations -> (none)
Changed lines of the file:
@@
 P 5390 5105
 F 0 "X1" H 5230 5375 50  0000 C CNN
-F 1 "ECS-2033-250-BN" H 5830 4840 50  0000 C CNN
+F 1 "OT3EL89CJI-111YLC-25M" H 5830 4840 50  0000 C CNN
 F 2 "RetroBitLab:OSC_ECS-2033-250-BN" H 5390 5105 50  0001 L BNN
-F 3 "https://www.lcsc.com/datasheet/C2441279.pdf" H 5390 5105 50  0001 L BNN
-F 4 "11/15/13" H 5390 5105 50  0001 L BNN "PARTREV"
-F 5 "ECS Inc" H 5390 5105 50  0001 L BNN "MANUFACTURER"
-F 6 "Manufacturer Recommendations" H 5390 5105 50  0001 L BNN "STANDARD"
-F 7 "C2441279" H 5390 5105 50  0001 C CNN "LCSC"
+F 3 "https://www.lcsc.com/datasheet/C7471623.pdf" H 5390 5105 50  0001 L BNN
+F 4 "YXC" H 5390 5105 50  0001 L BNN "MANUFACTURER"
+F 5 "C7471623" H 5390 5105 50  0001 C CNN "LCSC"
 	1    5390 5105
 	1    0    0    -1
